File: miscellaneous.kicad_sch (KiCad schematic)
At the start: 10 parts, among them SW7001 SW_MEC_5E, SW7002 SW_MEC_5E, SW7003 SW_MEC_5E, SW7004 SW_MEC_5E

Commit message: Fixed MGM240P pinout, replaced 01x06 SPI and UART header pins with 02x06 header pins that will be connected via jumper shunts, deleted MMC1 (microSD)
Connections:
- net MGM_PA08 renamed MGM_PB01
Changed lines of the file:
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@@
 		)
 	)
-	(global_label "MGM_PA08"
+	(global_label "MGM_PB01"
 		(shape input)
 		(at 64.77 73.66 180)
@@
 		)
 		(property "Intersheetrefs" "${INTERSHEET_REFS}"
-			(at 51.8668 73.66 0)
+			(at 51.6854 73.66 0)
 			(effects
 				(font
